Commit message: First mapping test: - Improved performance in simulation by removing sonar - Changed D435 for D415 in simulation since costmap bugged - Modified .yaml files for costmap for debugging - Removed old meshes files

File: paul/paul_description/urdf/paul.gazebo.xacro (robot description, xacro)
@@ -15,6 +15,5 @@
       <publishTf>1</publishTf>
       <publishOdomTF>true</publishOdomTF>
-      <odometrySource>1</odometrySource>
-      <publish_odom>1</publish_odom>
+      <odometrySource>world</odometrySource>   <!-- options: encoder, world-->
       <publishWheelJointState>false</publishWheelJointState>
       <alwaysOn>true</alwaysOn>

File: paul/paul_description/urdf/paul.urdf.xacro (robot description, xacro)
@@ -76,4 +76,5 @@
   <xacro:include filename="$(find paul_description)/urdf/sensors/d435/_d435.urdf.xacro"/>
   <xacro:include filename="$(find paul_description)/urdf/sensors/sonar/sonar.urdf.xacro"/>
+  <xacro:include filename="$(find paul_description)/urdf/sensors/realsense_d415.urdf.xacro"/>
   <!-- ============================================== -->
   <!-- ==================== BASE ==================== -->
@@ -156,16 +157,23 @@
     <origin xyz="0.50614 0 0.1" rpy="0 0 0" />
   </xacro:lidar>
-  <!-- D435 RGB-D Sensor -->
-  <xacro:sensor_d435 parent="base_link" use_nominal_extrinsics="${use_nominal_extrinsics}" name="realsense" topics_ns="realsense">
-    <origin xyz="${realsense_pose_x} ${realsense_pose_y} ${realsense_pose_z}" rpy="${realsense_rot_x} ${realsense_rot_y} ${realsense_rot_z}"/>
-  </xacro:sensor_d435>
-  <!-- Sonars -->
-  <xacro:sonar name="left" parent="base_link">
+  <!-- D435 RGB-D Sensor, D415 in simulation for better performance with rtabmap in simulation -->
+  <xacro:if value="$(arg sim)">
+    <xacro:realsense_d415_sensor parent="base_link" name="realsense" >
+      <origin xyz="${realsense_pose_x} ${realsense_pose_y} ${realsense_pose_z}" rpy="${realsense_rot_x} ${realsense_rot_y} ${realsense_rot_z}"/>
+    </xacro:realsense_d415_sensor>
+  </xacro:if>
+  <xacro:unless value="$(arg sim)">
+    <xacro:sensor_d435 parent="base_link" use_nominal_extrinsics="${use_nominal_extrinsics}" name="realsense" topics_ns="realsense">
+      <origin xyz="${realsense_pose_x} ${realsense_pose_y} ${realsense_pose_z}" rpy="${realsense_rot_x} ${realsense_rot_y} ${realsense_rot_z}"/>
+    </xacro:sensor_d435>
+  </xacro:unless>
+  <!-- Sonars: currently commented for better performance with rtabmap in simulation -->
+  <xacro:sonar name="left" parent="base_link" enabled="false">
     <origin xyz="${base_width} 0.1 ${base_height - 0.2}" rpy="0 0 0"/>
   </xacro:sonar>
-  <xacro:sonar name="center" parent="base_link">
+  <xacro:sonar name="center" parent="base_link" enabled="false">
     <origin xyz="${base_width} 0 ${base_height - 0.2}" rpy="0 0 0"/>
   </xacro:sonar>
-  <xacro:sonar name="right" parent="base_link">
+  <xacro:sonar name="right" parent="base_link" enabled="false">
     <origin xyz="${base_width} -0.1 ${base_height - 0.2}" rpy="0 0 0"/>
   </xacro:sonar>

File: paul/paul_description/urdf/sensors/d435/_d435.gazebo.xacro (robot description, xacro)
@@ -37,5 +37,5 @@
           <clip>
             <near>0.1</near>
-            <far>100</far>
+            <far>3</far>
           </clip>
           <noise>
@@ -53,11 +53,11 @@
           <horizontal_fov>${85.2*deg_to_rad}</horizontal_fov>
           <image>
-            <width>1280</width>
-            <height>720</height>
+            <width>640</width>
+            <height>480</height>
             <format>L_INT8</format>
           </image>
           <clip>
             <near>0.1</near>
-            <far>100</far>
+            <far>3</far>
           </clip>
           <noise>
@@ -75,11 +75,11 @@
           <horizontal_fov>${85.2*deg_to_rad}</horizontal_fov>
           <image>
-            <width>1280</width>
-            <height>720</height>
+            <width>640</width>
+            <height>480</height>
             <format>L_INT8</format>
           </image>
           <clip>
             <near>0.1</near>
-            <far>100</far>
+            <far>3</far>
           </clip>
           <noise>
@@ -97,10 +97,10 @@
           <horizontal_fov>${85.2*deg_to_rad}</horizontal_fov>
           <image>
-            <width>1280</width>
-            <height>720</height>
+            <width>640</width>
+            <height>480</height>
           </image>
           <clip>
             <near>0.1</near>
-            <far>100</far>
+            <far>3</far>
           </clip>
           <noise>

File: paul/paul_description/urdf/sensors/lidar.urdf.xacro (robot description, xacro)
@@ -47,5 +47,5 @@
                 <plugin name="laser_node" filename="libgazebo_ros_laser.so">
                     <topicName>/laser_scan</topicName>
-                    <frameName>/laser_link</frameName> <!-- slash required for global namespace -->
+                    <frameName>laser_link</frameName> <!-- slash required for global namespace -->
                 </plugin>
             </sensor>

File: paul/paul_description/urdf/sensors/sonar/sonar.gazebo.xacro (robot description, xacro)
@@ -8,9 +8,9 @@
                 <pose>0 0 0 0 0 0</pose>
                 <visualize>false</visualize>
-                <update_rate>10</update_rate>
+                <update_rate>5</update_rate>
                 <ray>
                     <scan>
                         <horizontal>
-                            <samples>720</samples>
+                            <samples>2</samples>
                             <resolution>1</resolution>
                             <min_angle>-0.261799</min_angle> <!-- - 7.5 deg -->
@@ -37,5 +37,5 @@
                     <frameName>${reference_link}</frameName>
                     <radiation>ultrasound</radiation>
-                    <updateRate>10</updateRate>
+                    <updateRate>5</updateRate>
                     <fov>0.05</fov>
                     <gaussianNoise>0.0</gaussianNoise>

File: paul/paul_description/urdf/sensors/sonar/sonar.urdf.xacro (robot description, xacro)
@@ -3,5 +3,5 @@
   <!-- Includes -->
   <xacro:include filename="$(find paul_description)/urdf/sensors/sonar/sonar.gazebo.xacro"/>
-  <xacro:macro name="sonar" params="parent *origin name:=sonar topics_ns:=sonars">
+  <xacro:macro name="sonar" params="parent *origin name:=sonar topics_ns:=sonars enabled">
     <xacro:property name="M_PI" value="3.1415926535897931" />
     <xacro:property name="sonar_width" value="0.04"/>
@@ -24,5 +24,7 @@
     </joint>
     <!-- Sonar Gazebo Plugin -->
-    <xacro:gazebo_sonar sonar_name="${name}" reference_link="${name}_sonar_link" topics_ns="${topics_ns}"/>
+    <xacro:if value="${enabled}">
+        <xacro:gazebo_sonar sonar_name="${name}" reference_link="${name}_sonar_link" topics_ns="${topics_ns}"/>
+    </xacro:if>
   </xacro:macro>
 </robot>
